Commit message: Fix concave collision

File: URDF/kendama_ball/kendama_ball.urdf (robot description, URDF)
Before this commit: robot kendama_ball, 1 links, 0 joints
Links:
- link base_link: mass 0.08210370012115252 -> 0.07415529686232127; geometry collision mesh filename=meshes/kendama_ball.obj scale=0.001 0.001 0.001; visual mesh filename=meshes/kendama_ball.obj scale=0.001 0.001 0.001

File: URDF/kendama_hand/kendama_hand.urdf (robot description, URDF)
Before this commit: robot kendama_hand, 1 links, 0 joints
Links:
- link base_link: geometry collision mesh filename=meshes/kendama_hand.obj scale=0.001 0.001 0.001; visual mesh filename=meshes/kendama_hand.obj scale=0.001 0.001 0.001

Commit message: Merged julien with reward

File: URDF/kendama_ball/kendama_ball.urdf (robot description, URDF)
Before this commit: robot ballcustom3, 1 links, 0 joints
Links:
- link base_link: mass 0.07415529686232127 -> 0.08210370012115252; geometry collision mesh filename=meshes/base_link.stl scale=0.0015 0.0015 0.0015; visual mesh filename=meshes/base_link.stl scale=0.0015 0.0015 0.0015

File: URDF/kendama_hand/kendama_hand.urdf (robot description, URDF)
Before this commit: robot kendama_hand, 1 links, 0 joints
Links:
- link base_link: geometry collision mesh filename=meshes/base_link.obj scale=0.001 0.001 0.001; visual mesh filename=meshes/base_link.obj scale=0.001 0.001 0.001
