Commit message: Constraints

File: URDF/kendama_hand/kendama_hand.urdf (robot description, URDF)
Before this commit: robot kendama_hand, 1 links, 0 joints
Links:
- link base_link: mass 0.07681894886302162 -> 0.038818904886302162

Commit message: Revert "Merge remote-tracking branch 'origin/alexis' into main"
This reverts commit 9598da060570dee8d41f20312d9bba7891ea5eac.

File: URDF/kendama_hand/kendama_hand.urdf (robot description, URDF)
Before this commit: robot kendama_hand, 1 links, 0 joints
Links:
- link base_link: geometry collision mesh filename=meshes/kendama_hand.obj scale=0.001 0.001 0.001; visual mesh filename=meshes/kendama_hand.obj scale=0.001 0.001 0.001
