Commit message: Auto stash before merge of "main" and "origin/alexis"

File: URDF/cube/cube.urdf (robot description, URDF)
Before this commit: robot cube, 1 links, 0 joints
Links:
- link baseLink: mass 0.038818904886302162 -> 0.000001

File: URDF/kendama_hand/kendama_hand.urdf (robot description, URDF)
Before this commit: robot kendama_hand, 1 links, 0 joints
Links:
- link base_link: mass 0.038818904886302162 -> 0.077

Commit message: First working for training

File: URDF/cube/cube.urdf (robot description, URDF)
Before this commit: robot cube, 1 links, 0 joints
Links:
- link baseLink: mass 0.000001 -> 0.0388

File: URDF/kendama_hand/kendama_hand.urdf (robot description, URDF)
Before this commit: robot kendama_hand, 1 links, 0 joints
Links:
- link base_link: mass 0.077 -> 0.0388
